Commit message: link명 수정

File: simulation/kobuki.urdf.xacro (robot description, xacro)
@@ -11,5 +11,5 @@
   <!-- Kobuki -->
   <xacro:macro name="kobuki">
-  <link name="rplidar_link">
+  <link name="laser">
 		<collision>
 			<origin xyz="0 0 0" rpy="0 0 0"/>
@@ -30,11 +30,11 @@
 			<inertia ixx="1e-6" ixy="0" ixz="0" iyy="1e-6" iyz="0" izz="1e-6"/>
 		</inertial>
-	</link>
-	<joint name="rplidar_joint" type="fixed">
-		<axis xyz="0 1 0"/>
-		<origin xyz="0 0 0.235" rpy="0 0 0 "/>
-		<parent link="base_link"/>
-		<child link="rplidar_link"/>
-	</joint>
+  </link>
+  <joint name="rplidar_joint" type="fixed">
+	<axis xyz="0 1 0"/>
+	<origin xyz="0 0 0.235" rpy="0 0 0 "/>
+	<parent link="base_link"/>
+	<child link="laser"/>
+  </joint>
     <link name="base_footprint"/>
     <!--

File: simulation/kobuki_gazebo.urdf.xacro (robot description, xacro)
@@ -2,5 +2,5 @@
 <robot name="kobuki_sim" xmlns:xacro="http://ros.org/wiki/xacro">
   <xacro:macro name="kobuki_sim">
-  <gazebo reference="rplidar_link">
+  <gazebo reference="laser">
 	<sensor type="gpu_ray" name="head_rplidar_sensor">
 		<pose>0 0 0 0 0 0</pose>
@@ -29,5 +29,5 @@
 		<plugin name="gazebo_ros_head_rplidar_controller" filename="libgazebo_ros_gpu_laser.so">
 			<topicName>/scan</topicName>
-			<frameName>rplidar_link</frameName>
+			<frameName>laser</frameName>
 		</plugin>
 	</sensor>
